File: LinearPS.kicad_pcb (KiCad board)
At the start: 2 copper layers, 100 x 100 mm, 102 parts, among them J1 Conn_01x03, J10 Conn_01x01, J11 Conn_01x01, J12 Conn_01x01, J14 Conn_01x01, J2 Conn_01x02, J3 Conn_01x04, J4 Conn_01x01, J5 Conn_01x01, J6 Conn_01x01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

Commit message: upgrade to Kicad_599
Other:
- net class Default removed
