File: LinearPS.kicad_sch (KiCad schematic)
At the start: 102 parts, among them J1 Conn_01x03, J10 Conn_01x01, J11 Conn_01x01, J12 Conn_01x01, J14 Conn_01x01, J2 Conn_01x02, J3 Conn_01x04, J4 Conn_01x01, J5 Conn_01x01, J6 Conn_01x01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

Commit message: Update LinearPS.kicad_sch
Parts:
- C1, C10: Part_Number (none) -> EKM478M1HL40RRSAP
- C12, C2, C3, C7: Part_Number (none) -> EGS475M2GF12RRSAP
- C13, C14, C16, C4: Part_Number (none) -> S104ZYFE072L
- C15, C6, C9: Part_Number (none) -> T101KCHE062L
- C5: Part_Number (none) -> S224ZYFE082LF
- C8: Part_Number (none) -> H331KYAE052A-T
- D10: Part_Number (none) -> 1N4740ATA-TC/ON
- D11: Part_Number (none) -> 1N4004-JJ
- D12, D21: Part_Number (none) -> TOL-30BHRADAA
- D22: Part_Number (none) -> 1N4733ATA-TC/ON
- D23, D5, D6, D7, D9: Part_Number (none) -> PH1N4148TB
- D8: Part_Number (none) -> 1N4734A-TAP
- Q1: Part_Number (none) -> 2N3904TA
- Q2, Q4, Q5, Q6, Q7: Part_Number (none) -> TIP41C
- Q3: Part_Number (none) -> 2N3906TA
- R1, R19, R30, R9: Part_Number (none) -> R 2k2 1/4W 5%
- R10, R23, R37, R39: Part_Number (none) -> R 100k 1/4W 5%
- R11, R8: Part_Number (none) -> R 27k 1/4W 5%
- R12: Part_Number (none) -> R 56k 1/4W 5%
- R13: Part_Number (none) -> R 22k 1/4W 5%
- R14: Part_Number (none) -> R 1k 1/4W 5%
- R15, R20, R21, R28, R29, R34, R36, R38, R5, R6: Part_Number (none) -> R 10k 1/4W 5%
- R16, R32, R33: Part_Number (none) -> R 1k 1W 5%
- R17: Part_Number (none) -> R 33R 1/4W 5%
- R18: Part_Number (none) -> R 33k 1/4W 5%
- R2: Part_Number (none) -> R 82E 1W 5%
- R22, R31: Part_Number (none) -> R 3k9 1/4W 5%
- R24, R25, R26, R27, R7: Part_Number (none) -> R 0R47 5W 5%
- R3: Part_Number (none) -> R 220E 1W 5%
- R35: Part_Number (none) -> R 1M 1/4W 5%
- R4: Part_Number (none) -> R 4k7 1/4W 5%
- R40: Part_Number (none) -> R 47k 1/4W 5%
- RV1, RV2: Part_Number (none) -> Volume 10kB
- RV3: Part_Number (none) -> 3296W-1-104LF
- RV6: Part_Number (none) -> 3296W-1-203LF
- U1, U2, U3: Part_Number (none) -> LM358P
